Commit message: A2

File: src/my_ur3_description/robots/common.gazebo.xacro (robot description, xacro)
@@ -2,5 +2,7 @@
 <robot xmlns:xacro="http://ros.org/wiki/xacro">
   <gazebo>
-    <!-- Add your code here -->
+    <plugin name="gazebo_ros_control" filename="libgazebo_ros_control.so">
+        <robotNamespace>/ur3</robotNamespace>
+    </plugin>
   </gazebo>
 </robot>

File: src/my_ur3_description/robots/ur.transmission.xacro (robot description, xacro)
@@ -2,4 +2,14 @@
 <robot xmlns:xacro="http://ros.org/wiki/xacro">
   <xacro:macro name="ur_arm_transmission" params="prefix">
+<transmission name="tran1">
+    <type>transmission_interface/SimpleTransmission</type>
+    <joint name="${prefix}shoulder_pan_joint">
+        <hardwareInterface>EffortJointInterface</hardwareInterface>
+    </joint>
+    <actuator name="motor1">
+        <hardwareInterface>EffortJointInterface</hardwareInterface>
+        <mechanicalReduction>1</mechanicalReduction>
+    </actuator>
+</transmission>
     <!-- Add controller transmissions here -->
   </xacro:macro>
